File: hardware/main/main.kicad_pcb (KiCad board)
At the start: 2 copper layers, 41.5 x 41.5 mm, 11 parts, among them J1 61729-1010BLF, J2 FLASH, U1 ATtiny402-SS, U2 CH330N, U3 A3144EUA-T-JSM

Commit message: final pcb version
Parts:
- moved HALL 4.78 mm to (149.4, 73.2)
- moved J1 1.98 mm to (168.0, 55.2)
- renumbered U1 to ATtiny402-SS, J2 to FLASH, U3 to HALL
Routing:
- net GND: track 36.7 -> 41.4 mm
- net OUT: track 34.8 -> 39.5 mm
- net VCC: track 47.7 -> 50.0 mm
- net D-: track 18.8 -> 16.9 mm
- net D+: track 31.6 -> 30.7 mm
Other:
- board text added: "Rev V1.0 RPM By azaslavskis"

Commit message: added holdes
Routing:
- net GND: vias 3 -> 7
Changed lines of the file:
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@@
+	)
+	(via
+		(at 154.3 82.44)
+		(size 2.5)
+		(drill 3)
+		(layers "F.Cu" "B.Cu")
+		(free yes)
+		(net 1)
+	)
+	(via
+		(at 184.48 69.46)
+		(size 2.5)
+		(drill 3)
+		(layers "F.Cu" "B.Cu")
+		(free yes)
+		(net 1)
+	)
+	(via
+		(at 179.06 84.69)
+		(size 2.5)
+		(drill 3)
+		(layers "F.Cu" "B.Cu")
+		(free yes)
+		(net 1)
+	)
+	(via
+		(at 167.8 54)
+		(size 2.5)
+		(drill 3)
+		(layers "F.Cu" "B.Cu")
+		(free yes)
+		(net 1)
 	)
 	(via

Commit message: final version
Parts:
- added G***: LOGO, LOGO, B.Cu at (169.2, 69.0)
